File: PCB/Amplificatore/Amplificatore.sch (KiCad schematic (older format))
At the start: 15 parts

Commit message: Add files via upload
Parts:
- removed C?: 470pF, 250V, Capacitor_SMD:C_1210_3225Metric, symbol Device:C
- removed J?: AudioJack2_Switch, Connector_Audio:Jack_6.35mm_Neutrik_NMJ4HCD2_Horizontal, symbol Connector:AudioJack2_Switch
- removed R? (x3): 1Meg, Resistor_SMD:R_0805_2012Metric, symbol Device:R_Small_US
- removed R? (x2): 68K, Resistor_SMD:R_0805_2012Metric, symbol Device:R_Small_US
- removed R? (x2): 820R, Resistor_SMD:R_0805_2012Metric, symbol Device:R_Small_US
- removed R? (x2): 10K, 1/4W, Resistor_SMD:R_1210_3225Metric, symbol Device:R
- removed RV?: 20K, symbol Device:R_POT_Small
- removed SW?: SW_DPDT_x2, symbol Switch:SW_DPDT_x2
- removed U? (x2): ECC83, Valve:Valve_ECC-83-2, symbol Valve:ECC83
- added C1: 47nF, Capacitor_THT:C_Rect_L4.6mm_W3.0mm_P2.50mm_MKS02_FKP02, symbol Device:C
- added C2: 680nF, Capacitor_THT:C_Rect_L18.0mm_W11.0mm_P15.00mm_FKS3_FKP3, symbol Device:C
- added C3, C4: 22uF, Capacitor_THT:CP_Radial_D13.0mm_P5.00mm, symbol Device:CP
- added C5: 47pF, Capacitor_THT:C_Rect_L7.2mm_W4.5mm_P5.00mm_FKS2_FKP2_MKS2_MKP2, symbol Device:C
- added R1: 1Meg, Resistor_SMD:R_0805_2012Metric, symbol Device:R_Small_US
- added R2: 68K, Resistor_SMD:R_0805_2012Metric, symbol Device:R_Small_US
- added R3: 100K, Resistor_SMD:R_2512_6332Metric, symbol Device:R
- added R4: 2K7, Resistor_SMD:R_0805_2012Metric, symbol Device:R_Small_US
- added R5: 10K, Resistor_SMD:R_2512_6332Metric, symbol Device:R
- added U2: ECC83, Valve:Valve_ECC-83-2, symbol Valve:ECC83
Connections:
- wire segments 27 -> 29

Commit message: avanzamento pcb
Parts:
- added C10: 680nF, Capacitor_THT:C_Rect_L18.0mm_W11.0mm_P15.00mm_FKS3_FKP3, symbol Device:C
- added C11, C5: 22nF, Capacitor_THT:C_Rect_L13.0mm_W4.0mm_P10.00mm_FKS3_FKP3_MKS4, symbol Device:C
- added C7: 1nF, Capacitor_THT:C_Rect_L13.0mm_W4.0mm_P10.00mm_FKS3_FKP3_MKS4, symbol Device:C
- added C8: 10uF, Capacitor_Tantalum_SMD:CP_EIA-3216-10_Kemet-I, symbol Device:CP
- added C9: 470pF, Capacitor_THT:C_Rect_L10.0mm_W3.0mm_P7.50mm_MKS4, symbol Device:C
- added J1: POT-1, Connector_PinSocket_2.00mm:PinSocket_1x03_P2.00mm_Vertical, symbol Connector_Generic:Conn_01x03
- added R6, R8: 100K, Resistor_SMD:R_2512_6332Metric, symbol Device:R
- added R7: 1K5, Resistor_SMD:R_0805_2012Metric, symbol Device:R_Small_US
- added R9: 47K, Resistor_SMD:R_2512_6332Metric, symbol Device:R
- added unit 2 of U1
- renumbered C3 to C2, C5 to C3, C2 to C4, C4 to C6, R4 to R3, R3 to R4, U2 to U1
Connections:
- net GND: now also C10.1, C8.2, J1.3 (Pin_3), R7.2
- net at C6.1, R5.1: now also R4.1, C9.2, R8.1
- net at C3.2, R4.2, U1.6 (A): now also C5.2
- net at C2.1, R5.2: no longer R4.1
- new net: C5.1, C7.2, J1.1 (Pin_1)
- new net: C7.1, J1.2 (Pin_2), R6.2
- new net: R6.1, U1.2 (G)
- new net: C11.2, C9.1, R8.2, U1.1 (A)
- new net: C10.2, C8.1, R7.1, U1.3 (K)
- new net: C11.1, R9.2
Other:
- moved on the sheet: C2, C6, R5

Commit message: Add files via upload
Parts:
- added D? (x3): 1N4007, Diode_THT:D_DO-41_SOD81_P10.16mm_Horizontal, symbol Diode:1N4007
- added K1: G5Q-1, Relay_THT:Relay_SPDT_Omron-G5Q-1, symbol Relay:G5Q-1
- added R10, R11: 220K, Resistor_SMD:R_2512_6332Metric, symbol Device:R
- J1: PN 292161-3 -> 1-292161-3
Connections:
- net at R6.1, U1.2 (G): now also R10.2
- net at C11.1, R9.2: now also R11.1
- net at R9.1: now also K1.3
- new net: D?.1 (K), D?.2 (A), K1.2
- new net: K1.4, R10.1, R11.2
- new net: D?.1 (K), D?.2 (A) (x2)
- new net LEAD-SW-A: K1.1
- new net LEAD-SW-B: K1.5
Changed lines of the file:
@@
 F 2 "Connector_PinSocket_2.00mm:PinSocket_1x03_P2.00mm_Vertical" H 4350 3900 50  0001 C CNN
 F 3 "~" H 4350 3900 50  0001 C CNN
-F 4 "292161-3" H 4350 3900 50  0001 C CNN "PN"
+F 4 "1-292161-3" H 4350 3900 50  0001 C CNN "PN"
 F 5 "M: 571-292161-3" H 4350 3900 50  0001 C CNN "FORNITORE"
 F 6 "AMP-CT, 2mm, Verticale, 3 Pin" H 4350 3900 50  0001 C CNN "NOTE"
@@
 $EndComp
 Wire Wire Line
-	5350 3900 5650 3900
+	5350 3900 5550 3900
 $Comp
 L Device:R_Small_US R7
@@
 	5350 2000 5950 2000
 Connection ~ 3200 2000
+Wire Wire Line
+	7100 3400 7100 3700
+Wire Wire Line
+	7100 3700 7700 3700
+$Comp
+L Relay:G5Q-1 K1
+U 1 1 610D4A05
+P 7400 3200
+F 0 "K1" V 7967 3200 50  0000 C CNN
+F 1 "G5Q-1" V 7876 3200 50  0000 C CNN
+F 2 "Relay_THT:Relay_SPDT_Omron-G5Q-1" H 7850 3150 50  0001 L CNN
+F 3 "https://www.omron.com/ecb/products/pdf/en-g5q.pdf" H 7400 3200 50  0001 L CNN
+F 4 "G5Q-1 DC6 " V 7400 3200 50  0001 C CNN "PN"
+F 5 "M: 653-G5Q-1DC6 " V 7400 3200 50  0001 C CNN "FORNITORE"
+	1    7400 3200
+	0    -1   -1   0
+$EndComp
+Text GLabel 7700 3400 2    50   Input ~ 0
+LEAD-SW-A
+Text GLabel 7700 3700 2    50   Input ~ 0
+LEAD-SW-B
+Connection ~ 6850 2900
+$Comp
+L Device:R R11
+U 1 1 610E3F3A
+P 6850 3200
+F 0 "R11" H 6920 3246 50  0000 L CNN
+F 1 "220K" H 6920 3155 50  0000 L CNN
+F 2 "Resistor_SMD:R_2512_6332Metric" V 6780 3200 50  0001 C CNN
+F 3 "~" H 6850 3200 50  0001 C CNN
+F 4 "CRCW2512220KJNEG " H 6850 3200 50  0001 C CNN "PN"
+F 5 "M: 71-CRCW2512J-220K-E3 " H 6850 3200 50  0001 C CNN "FORNITORE"
+F 6 "1W, 5%, 500VDC" H 6850 3200 50  0001 C CNN "NOTE"
+	1    6850 3200
+	-1   0    0    -1
+$EndComp
+$Comp
+L Device:R R10
+U 1 1 610E4EA1
+P 5550 3550
+F 0 "R10" H 5620 3596 50  0000 L CNN
+F 1 "220K" H 5620 3505 50  0000 L CNN
+F 2 "Resistor_SMD:R_2512_6332Metric" V 5480 3550 50  0001 C CNN
+F 3 "~" H 5550 3550 50  0001 C CNN
+F 4 "CRCW2512220KJNEG " H 5550 3550 50  0001 C CNN "PN"
+F 5 "M: 71-CRCW2512J-220K-E3 " H 5550 3550 50  0001 C CNN "FORNITORE"
+F 6 "1W, 5%, 500VDC" H 5550 3550 50  0001 C CNN "NOTE"
+	1    5550 3550
+	-1   0    0    -1
+$EndComp
+Wire Wire Line
+	5550 3700 5550 3900
+Connection ~ 5550 3900
+Wire Wire Line
+	5550 3900 5650 3900
+Wire Wire Line
+	5550 3400 6850 3400
+Wire Wire Line
+	6850 3400 6850 3350
+Wire Wire Line
+	6850 3050 6850 2900
+Wire Wire Line
+	6850 3400 7000 3400
+Wire Wire Line
+	7000 3400 7000 3100
+Wire Wire Line
+	7000 3100 7100 3100
+Connection ~ 6850 3400
+Wire Wire Line
+	7100 2900 7000 2900
+Wire Wire Line
+	7000 2900 7000 2150
+Wire Wire Line
+	7000 2150 6850 2150
+Wire Wire Line
+	6850 2150 6850 2350
+$Comp
+L Diode:1N4007 D?
+U 1 1 611044D8
+P 7900 2750
+F 0 "D?" V 7946 2830 50  0000 L CNN
+F 1 "1N4007" V 7855 2830 50  0000 L CNN
+F 2 "Diode_THT:D_DO-41_SOD81_P10.16mm_Horizontal" H 7900 2575 50  0001 C CNN
+F 3 "http://www.vishay.com/docs/88503/1n4001.pdf" H 7900 2750 50  0001 C CNN
+F 4 "1N4007-T" H 7900 2750 50  0001 C CNN "PN"
+F 5 "M: 621-1N4007 " H 7900 2750 50  0001 C CNN "FORNITORE"
+	1    7900 2750
+	0    1    -1   0
+$EndComp
+$Comp
+L Diode:1N4007 D?
+U 1 1 6110AC70
+P 7900 2250
+F 0 "D?" V 7946 2330 50  0000 L CNN
+F 1 "1N4007" V 7855 2330 50  0000 L CNN
+F 2 "Diode_THT:D_DO-41_SOD81_P10.16mm_Horizontal" H 7900 2075 50  0001 C CNN
+F 3 "http://www.vishay.com/docs/88503/1n4001.pdf" H 7900 2250 50  0001 C CNN
+F 4 "1N4007-T" H 7900 2250 50  0001 C CNN "PN"
+F 5 "M: 621-1N4007 " H 7900 2250 50  0001 C CNN "FORNITORE"
+	1    7900 2250
+	0    1    -1   0
+$EndComp
+Wire Wire Line
+	7900 2600 7900 2400
+$Comp
+L Diode:1N4007 D?
+U 1 1 6110D37C
+P 8400 2750
+F 0 "D?" V 8354 2830 50  0000 L CNN
+F 1 "1N4007" V 8445 2830 50  0000 L CNN
+F 2 "Diode_THT:D_DO-41_SOD81_P10.16mm_Horizontal" H 8400 2575 50  0001 C CNN
+F 3 "http://www.vishay.com/docs/88503/1n4001.pdf" H 8400 2750 50  0001 C CNN
+F 4 "1N4007-T" H 8400 2750 50  0001 C CNN "PN"
+F 5 "M: 621-1N4007 " H 8400 2750 50  0001 C CNN "FORNITORE"
+	1    8400 2750
+	0    1    1    0
+$EndComp
+Wire Wire Line
+	7900 2900 7900 3000
+Wire Wire Line
+	7900 3000 8400 3000
+Wire Wire Line
+	8400 3000 8400 2900
+Wire Wire Line
+	8400 2600 8400 2050
+Wire Wire Line
+	8400 2050 7900 2050
+Wire Wire Line
+	7900 2050 7900 2100
+Wire Wire Line
+	7700 3000 7900 3000
+Connection ~ 7900 3000
 $EndSCHEMATC

Commit message: ...
Parts:
- added C12: 1nF, Capacitor_THT:C_Rect_L13.0mm_W4.0mm_P10.00mm_FKS3_FKP3_MKS4, symbol Device:C
- added C13, C22: 2n2F, Capacitor_THT:C_Rect_L13.0mm_W4.0mm_P10.00mm_FKS3_FKP3_MKS4, symbol Device:C
- added C14, C15, C16, C21: 100nF, Capacitor_THT:C_Rect_L18.0mm_W5.0mm_P15.00mm_FKS3_FKP3, symbol Device:C
- added C17: 4n7F, Capacitor_THT:C_Rect_L13.0mm_W4.0mm_P10.00mm_FKS3_FKP3_MKS4, symbol Device:C
- added C18: 10nF, Capacitor_THT:C_Rect_L13.0mm_W4.0mm_P10.00mm_FKS3_FKP3_MKS4, symbol Device:C
- added C19: 220pF, Capacitor_THT:C_Rect_L7.2mm_W4.5mm_P5.00mm_FKS2_FKP2_MKS2_MKP2, symbol Device:C
- added C20: 470pF, Capacitor_THT:C_Rect_L10.0mm_W3.0mm_P7.50mm_MKS4, symbol Device:C
- added D1, D4, D6, D7: 1N4007, Diode_THT:D_DO-41_SOD81_P10.16mm_Horizontal, symbol Diode:1N4007
- added J10: POWER, Connector_Molex:Molex_KK-396_A-41791-0003_1x03_P3.96mm_Vertical, symbol Connector_Generic:Conn_01x03
- added J11: FILAMENT-U2, Connector_PinSocket_2.00mm:PinSocket_1x03_P2.00mm_Vertical, symbol Connector_Generic:Conn_01x03
- added J12: FILAMENT-U1, Connector_PinSocket_2.00mm:PinSocket_1x03_P2.00mm_Vertical, symbol Connector_Generic:Conn_01x03
- added J2: POT-LEAD, Connector_PinSocket_2.00mm:PinSocket_1x03_P2.00mm_Vertical, symbol Connector_Generic:Conn_01x03
- added J3: SEND-RETURN, Connector_PinSocket_2.00mm:PinSocket_1x03_P2.00mm_Vertical, symbol Connector_Generic:Conn_01x03
- added J4: In, Connector_PinSocket_2.00mm:PinSocket_1x03_P2.00mm_Vertical, symbol Connector_Generic:Conn_01x03
- added J5: POT-BASS-BACK, Connector_PinSocket_2.00mm:PinSocket_1x03_P2.00mm_Vertical, symbol Connector_Generic:Conn_01x03
- added J6: POT-MID, Connector_PinSocket_2.00mm:PinSocket_1x03_P2.00mm_Vertical, symbol Connector_Generic:Conn_01x03
- added J7: POT-TREBLE, Connector_PinSocket_2.00mm:PinSocket_1x03_P2.00mm_Vertical, symbol Connector_Generic:Conn_01x03
- added J8: POT-BASS-FRONT, Connector_PinSocket_2.00mm:PinSocket_1x03_P2.00mm_Vertical, symbol Connector_Generic:Conn_01x03
- added J9: MASTER, Connector_PinSocket_2.00mm:PinSocket_1x03_P2.00mm_Vertical, symbol Connector_Generic:Conn_01x03
- added K2, K3, K4: G5Q-1, Relay_THT:Relay_SPDT_Omron-G5Q-1, symbol Relay:G5Q-1
- added R12, R20, R27: 10K, Resistor_SMD:R_2512_6332Metric, symbol Device:R
- added R13, R17, R19, R25, R26, R28: 100K, Resistor_SMD:R_2512_6332Metric, symbol Device:R
- added R14, R18: 47K, Resistor_SMD:R_2512_6332Metric, symbol Device:R
- added R15, R22: 1Meg, Resistor_SMD:R_0805_2012Metric, symbol Device:R_Small_US
- added R16: 1K5, Resistor_SMD:R_0805_2012Metric, symbol Device:R_Small_US
- added R21: 10R, Resistor_SMD:R_2512_6332Metric, symbol Device:R
- added R23: 470R, Resistor_SMD:R_0805_2012Metric, symbol Device:R_Small_US
- added R24: 220K, Resistor_SMD:R_2512_6332Metric, symbol Device:R
- added unit 3 of U1
- added U2: ECC83, Valve:Valve_ECC-83-2, symbol Valve:ECC83
- J1: value POT-1 -> POT-GAIN
- gave numbers to parts that had none: 3
Connections:
- net GND: now also D3.1 (K), D5.2 (A), K1.2, C12.1, C13.1, C22.1, D6.1 (K), D7.2 (A), J10.3 (Pin_3), J2.3 (Pin_3), J4.3 (Pin_3), J6.3 (Pin_3), J8.3 (Pin_3), J9.3 (Pin_3), R16.2, R20.1, R21.1, R22.2, R23.2, R25.2
- net at C9.2, R4.1, R8.1: now also C2.1, R5.2; no longer C6.1, R5.1
- net Mute: now reaches C5.1, C7.2, J1.1 (Pin_1)
- net Mute: now also J4.2 (Pin_2)
- net at K1.3, R9.1: now also C12.2, D1.1 (K), D4.2 (A), J2.1 (Pin_1)
- net at K1.4, R10.1, R11.2: now also K2.3, R12.2
- net at D2.2 (A), D5.1 (K): now also D1.2 (A), D4.1 (K)
- net at C1.2: now also J4.1 (Pin_1)
- net LEAD-SW-A renamed LEAD-SW
- net LEAD-SW-B renamed COMMON
- net COMMON: now also K2.5, K3.5, K4.5
- new net: J2.2 (Pin_2), R14.2
- new net: R12.1, R13.2
- new net: R13.1, R14.1, R15.1, R18.1, U2.7 (G)
- new net: C14.2, R17.2, U2.6 (A)
- new net: R16.1, U2.8 (K)
- new net: C14.1, R15.2, R19.1
- new net: K3.2, R19.2, R20.2
- new net: C13.2, D6.2 (A), D7.1 (K), K2.2, R18.2
- new net: J3.3 (Pin_3), K3.3
- new net: K3.4, K4.4
- new net: J3.1 (Pin_1), K4.3
- new net: J3.2 (Pin_2), R21.2
- new net: C15.2, K4.2
- new net: C16.2, C17.2, C19.2, R24.2, R26.1, U2.1 (A)
- new net: R23.1, U2.3 (K)
- new net: C16.1, J5.1 (Pin_1)
- new net: C17.1, J5.2 (Pin_2)
- new net: J5.3 (Pin_3), R25.1
- new net: C18.2, C21.1, R26.2
- new net: C18.1, J6.2 (Pin_2)
- new net: C20.1, J6.1 (Pin_1)
- new net: C19.1, C20.2, J7.1 (Pin_1)
- new net: C21.2, R27.2
- new net: C22.2, J7.3 (Pin_3), R27.1, R28.1
- new net: J7.2 (Pin_2), J9.1 (Pin_1)
- new net: J8.1 (Pin_1), J8.2 (Pin_2), R28.2
- new net: J12.1 (Pin_1), U1.4 (F1)
- new net: J12.2 (Pin_2), U1.5 (F1)
- new net: J12.3 (Pin_3), U1.9 (F2)
- new net: J11.1 (Pin_1), U2.4 (F1)
- new net: J11.2 (Pin_2), U2.5 (F1)
- new net: J11.3 (Pin_3), U2.9 (F2)
- new net Earth: J10.2 (Pin_2)
- new net FILTRO_IN: C15.1, R22.1, U2.2 (G)
- new net RITHM-SW: K2.1
- new net SEND-SW: K3.1, K4.1
- new net VCC: C6.1, J10.1 (Pin_1), R17.1, R24.1, R5.1
Other:
- moved on the sheet: C2, C6, R5
